File: hardware/Iq Mixer.sch (KiCad schematic (older format))
At the start: 24 parts, among them IC1 LTC5598, P1 BNC, P2 BNC, P3 BNC, P4 BNC, T1 TRANSFO4, T2 TRANSFO4

Commit message: Footprint-association
Parts:
- C1, C2, C3, C6, C8: footprint (none) -> Capacitors_SMD:C_0603_HandSoldering
- C10, C9: renamed from C?; footprint (none) -> Capacitors_SMD:c_elec_5x5.3
- C11: renamed from C?; footprint (none) -> Capacitors_SMD:C_0603_HandSoldering
- C4, C5, C7: footprint (none) -> Capacitors_SMD:c_elec_5x5.3
- IC1: footprint (none) -> Housings_DFN_QFN:QFN-24-1EP_4x4mm_Pitch0.5mm
- JP1: footprint (none) -> Connect:PINHEAD1-3
- R1: footprint (none) -> Resistors_SMD:R_0603_HandSoldering
- U1: renamed from U?; footprint (none) -> TO_SOT_Packages_SMD:TO-263-3Lead
- W1, W2: renamed from W?; footprint (none) -> Wire_Pads:SolderWirePad_single_SMD_5x10mm
- gave numbers to parts that had none: 1
Changed lines of the file:
@@
 F 0 "IC1" H 6450 2650 60  0000 C CNN
 F 1 "LTC5598" H 5800 3250 60  0000 C CNN
-F 2 "" H 5750 3500 60  0001 C CNN
+F 2 "Housings_DFN_QFN:QFN-24-1EP_4x4mm_Pitch0.5mm" H 5750 3500 60  0001 C CNN
 F 3 "" H 5750 3500 60  0001 C CNN
 	1    5750 3500
@@
 F 0 "P4" H 7410 3820 50  0000 C CNN
 F 1 "BNC" V 7510 3640 50  0000 C CNN
-F 2 "" H 7400 3700 50  0000 C CNN
+F 2 "" H 7400 3700 50  0001 C CNN
 F 3 "" H 7400 3700 50  0000 C CNN
 	1    7400 3700
@@
 F 0 "C6" H 6975 3800 50  0000 L CNN
 F 1 "10nF" H 6975 3600 50  0000 L CNN
-F 2 "" H 6988 3550 50  0000 C CNN
+F 2 "Capacitors_SMD:C_0603_HandSoldering" H 6988 3550 50  0001 C CNN
 F 3 "" H 6950 3700 50  0000 C CNN
 	1    6950 3700
@@
 F 0 "C8" H 7175 3650 50  0000 L CNN
 F 1 "1nF" H 7175 3450 50  0000 L CNN
-F 2 "" H 7188 3400 50  0000 C CNN
+F 2 "Capacitors_SMD:C_0603_HandSoldering" H 7188 3400 50  0001 C CNN
 F 3 "" H 7150 3550 50  0000 C CNN
 	1    7150 3550
@@
 F 0 "C7" H 7175 3450 50  0000 L CNN
 F 1 "4,7uF" H 7175 3250 50  0000 L CNN
-F 2 "" H 7188 3200 50  0000 C CNN
+F 2 "Capacitors_SMD:c_elec_5x5.3" H 7188 3200 50  0001 C CNN
 F 3 "" H 7150 3350 50  0000 C CNN
 	1    7150 3350
@@
 F 0 "C4" H 5225 3100 50  0000 L CNN
 F 1 "4,7uF" H 5225 2900 50  0000 L CNN
-F 2 "" H 5238 2850 50  0000 C CNN
+F 2 "Capacitors_SMD:c_elec_5x5.3" H 5238 2850 50  0001 C CNN
 F 3 "" H 5200 3000 50  0000 C CNN
 	1    5200 3000
@@
 F 0 "C3" H 5025 3100 50  0000 L CNN
 F 1 "1nF" H 5025 2900 50  0000 L CNN
-F 2 "" H 5038 2850 50  0000 C CNN
+F 2 "Capacitors_SMD:C_0603_HandSoldering" H 5038 2850 50  0001 C CNN
 F 3 "" H 5000 3000 50  0000 C CNN
 	1    5000 3000
@@
 F 0 "C5" H 5225 4500 50  0000 L CNN
 F 1 "470nF" H 5225 4300 50  0000 L CNN
-F 2 "" H 5238 4250 50  0000 C CNN
+F 2 "Capacitors_SMD:c_elec_5x5.3" H 5238 4250 50  0001 C CNN
 F 3 "" H 5200 4400 50  0000 C CNN
 	1    5200 4400
@@
 F 0 "R1" V 4430 3850 50  0000 C CNN
 F 1 "50Ohm" V 4350 3850 50  0000 C CNN
-F 2 "" V 4280 3850 50  0000 C CNN
+F 2 "Resistors_SMD:R_0603_HandSoldering" V 4280 3850 50  0001 C CNN
 F 3 "" H 4350 3850 50  0000 C CNN
 	1    4350 3850
@@
 F 0 "C1" H 4725 3750 50  0000 L CNN
 F 1 "10nF" H 4725 3550 50  0000 L CNN
-F 2 "" H 4738 3500 50  0000 C CNN
+F 2 "Capacitors_SMD:C_0603_HandSoldering" H 4738 3500 50  0001 C CNN
 F 3 "" H 4700 3650 50  0000 C CNN
 	1    4700 3650
@@
 F 0 "P1" H 4060 3770 50  0000 C CNN
 F 1 "BNC" V 4160 3590 50  0000 C CNN
-F 2 "" H 4050 3650 50  0000 C CNN
+F 2 "" H 4050 3650 50  0001 C CNN
 F 3 "" H 4050 3650 50  0000 C CNN
 	1    4050 3650
@@
 F 0 "JP1" H 4400 3100 50  0000 L CNN
 F 1 "JUMPER3" H 4350 3300 50  0000 C BNN
-F 2 "" H 4350 3200 50  0000 C CNN
+F 2 "Connect:PINHEAD1-3" H 4350 3200 50  0001 C CNN
 F 3 "" H 4350 3200 50  0000 C CNN
 	1    4350 3200
@@
 F 0 "T1" H 5850 5450 50  0000 C CNN
 F 1 "TRANSFO4" H 5850 4900 50  0000 C CNN
-F 2 "" H 5850 5200 50  0000 C CNN
+F 2 "" H 5850 5200 50  0001 C CNN
 F 3 "" H 5850 5200 50  0000 C CNN
 	1    5850 5200
@@
 F 0 "P3" H 5960 6070 50  0000 C CNN
 F 1 "BNC" V 6060 5890 50  0000 C CNN
-F 2 "" H 5950 5950 50  0000 C CNN
+F 2 "" H 5950 5950 50  0001 C CNN
 F 3 "" H 5950 5950 50  0000 C CNN
 	1    5950 5950
@@
 F 0 "T2" H 5950 2550 50  0000 C CNN
 F 1 "TRANSFO4" H 5950 2000 50  0000 C CNN
-F 2 "" H 5950 2300 50  0000 C CNN
+F 2 "" H 5950 2300 50  0001 C CNN
 F 3 "" H 5950 2300 50  0000 C CNN
 	1    5950 2300
@@
 F 0 "P2" H 5910 1720 50  0000 C CNN
 F 1 "BNC" V 6010 1540 50  0000 C CNN
-F 2 "" H 5900 1600 50  0000 C CNN
+F 2 "" H 5900 1600 50  0001 C CNN
 F 3 "" H 5900 1600 50  0000 C CNN
 	1    5900 1600
@@
 $EndComp
 $Comp
-L C C?
+L C C11
 U 1 1 59FE30ED
 P 10700 3550
-F 0 "C?" H 10725 3650 50  0000 L CNN
+F 0 "C11" H 10725 3650 50  0000 L CNN
 F 1 "100nF" H 10725 3450 50  0000 L CNN
-F 2 "" H 10738 3400 50  0000 C CNN
+F 2 "Capacitors_SMD:C_0603_HandSoldering" H 10738 3400 50  0001 C CNN
 F 3 "" H 10700 3550 50  0000 C CNN
 	1    10700 3550
@@
 $EndComp
 $Comp
-L INDUCTOR L?
+L INDUCTOR L1
 U 1 1 59FE3170
 P 10400 3400
-F 0 "L?" V 10350 3400 50  0000 C CNN
+F 0 "L1" V 10350 3400 50  0000 C CNN
 F 1 "20uH" V 10500 3400 50  0000 C CNN
-F 2 "" H 10400 3400 50  0000 C CNN
+F 2 "" H 10400 3400 50  0001 C CNN
 F 3 "" H 10400 3400 50  0000 C CNN
 	1    10400 3400
@@
 $EndComp
 $Comp
-L 7805 U?
+L 7805 U1
 U 1 1 59FE3952
 P 9650 3450
-F 0 "U?" H 9800 3254 50  0000 C CNN
+F 0 "U1" H 9800 3254 50  0000 C CNN
 F 1 "7805" H 9650 3650 50  0000 C CNN
-F 2 "" H 9650 3450 50  0000 C CNN
+F 2 "TO_SOT_Packages_SMD:TO-263-3Lead" H 9650 3450 50  0001 C CNN
 F 3 "" H 9650 3450 50  0000 C CNN
 	1    9650 3450
@@
 $EndComp
 $Comp
-L C C?
+L C C10
 U 1 1 59FE3E8B
 P 10100 3550
-F 0 "C?" H 10125 3650 50  0000 L CNN
+F 0 "C10" H 10125 3650 50  0000 L CNN
 F 1 "1uF" H 10125 3450 50  0000 L CNN
-F 2 "" H 10138 3400 50  0000 C CNN
+F 2 "Capacitors_SMD:c_elec_5x5.3" H 10138 3400 50  0001 C CNN
 F 3 "" H 10100 3550 50  0000 C CNN
 	1    10100 3550
@@
 	8850 3700 10700 3700
 $Comp
-L GND #PWR?
+L GND #PWR014
 U 1 1 59FE43F2
 P 10100 3700
-F 0 "#PWR?" H 10100 3450 50  0001 C CNN
+F 0 "#PWR014" H 10100 3450 50  0001 C CNN
 F 1 "GND" H 10100 3550 50  0000 C CNN
 F 2 "" H 10100 3700 50  0000 C CNN
@@
 F 0 "C2" H 4725 3950 50  0000 L CNN
 F 1 "10nF" H 4725 3750 50  0000 L CNN
-F 2 "" H 4738 3700 50  0000 C CNN
+F 2 "Capacitors_SMD:C_0603_HandSoldering" H 4738 3700 50  0001 C CNN
 F 3 "" H 4700 3850 50  0000 C CNN
 	1    4700 3850
@@
 	4550 3850 4500 3850
 $Comp
-L VCC #PWR?
+L VCC #PWR015
 U 1 1 59FE4933
 P 10700 3350
-F 0 "#PWR?" H 10700 3200 50  0001 C CNN
+F 0 "#PWR015" H 10700 3200 50  0001 C CNN
 F 1 "VCC" H 10700 3500 50  0000 C CNN
 F 2 "" H 10700 3350 50  0000 C CNN
@@
 	10700 3350 10700 3400
 $Comp
-L C C?
+L C C9
 U 1 1 59FE4A8A
 P 9250 3550
-F 0 "C?" H 9275 3650 50  0000 L CNN
+F 0 "C9" H 9275 3650 50  0000 L CNN
 F 1 "1uF" H 9275 3450 50  0000 L CNN
-F 2 "" H 9288 3400 50  0000 C CNN
+F 2 "Capacitors_SMD:c_elec_5x5.3" H 9288 3400 50  0001 C CNN
 F 3 "" H 9250 3550 50  0000 C CNN
 	1    9250 3550
@@
 Connection ~ 9650 3700
 $Comp
-L TEST_1P W?
+L TEST_1P W1
 U 1 1 59FE4DB4
 P 8850 3400
-F 0 "W?" H 8850 3670 50  0000 C CNN
+F 0 "W1" H 8850 3670 50  0000 C CNN
 F 1 "VIN" H 8850 3600 50  0000 C CNN
-F 2 "" H 9050 3400 50  0000 C CNN
+F 2 "Wire_Pads:SolderWirePad_single_SMD_5x10mm" H 9050 3400 50  0001 C CNN
 F 3 "" H 9050 3400 50  0000 C CNN
 	1    8850 3400
@@
 $EndComp
 $Comp
-L TEST_1P W?
+L TEST_1P W2
 U 1 1 59FE4E36
 P 8850 3700
-F 0 "W?" H 8850 3970 50  0000 C CNN
+F 0 "W2" H 8850 3970 50  0000 C CNN
 F 1 "VGND" H 8850 3900 50  0000 C CNN
-F 2 "" H 9050 3700 50  0000 C CNN
+F 2 "Wire_Pads:SolderWirePad_single_SMD_5x10mm" H 9050 3700 50  0001 C CNN
 F 3 "" H 9050 3700 50  0000 C CNN
 	1    8850 3700

Commit message: Layout, Gerber
Parts:
- removed JP1: JUMPER3, Connect:PINHEAD1-3, symbol JUMPER3
- C4: value 4,7uF -> 100n; footprint Capacitors_SMD:c_elec_5x5.3 -> Capacitors_SMD:C_0603_HandSoldering
- C7: value 4,7uF -> 100nF; footprint Capacitors_SMD:c_elec_5x5.3 -> Capacitors_SMD:C_0603_HandSoldering
- L1: footprint (none) -> Resistors_SMD:R_0805_HandSoldering
- P1: value BNC -> SMA_LO; footprint (none) -> Molex_SMA:Molex_SMA_Jack_Edge_Mount
- P2: value BNC -> SMA_I; footprint (none) -> Molex_SMA:Molex_SMA_Jack_Edge_Mount
- P3: value BNC -> SMA_Q; footprint (none) -> Molex_SMA:Molex_SMA_Jack_Edge_Mount
- P4: value BNC -> SMA_OUT; footprint (none) -> Molex_SMA:Molex_SMA_Jack_Edge_Mount
- T1, T2: footprint (none) -> Balun:Balun
- U1: footprint TO_SOT_Packages_SMD:TO-263-3Lead -> TO_SOT_Packages_THT:TO-220_Neutral123_Vertical
Connections:
- net GND: now also T1.5 (S2), T2.2 (PM), T2.4 (S1); no longer T1.4 (S1), T2.5 (S2)
- net VCC: no longer T2.2 (PM)
- net at IC1.10 (BBPQ): now also T1.3 (PR2); no longer T1.1 (PR1)
- net at IC1.21 (BBPI): now also T2.1 (PR1); no longer T2.3 (PR2)
- net at IC1.22 (BBMI): now also T2.3 (PR2); no longer T2.1 (PR1)
- net at IC1.9 (BBMQ): now also T1.1 (PR1); no longer T1.3 (PR2)
- net at P3.1 (In): now also T1.4 (S1); no longer T1.5 (S2)
- net at P2.1 (In): now also T2.5 (S2); no longer T2.4 (S1)
- no-connect marks 0 -> 1
Other:
- moved on the sheet: T1
Changed lines of the file:
@@
 P 7400 3700
 F 0 "P4" H 7410 3820 50  0000 C CNN
-F 1 "BNC" V 7510 3640 50  0000 C CNN
-F 2 "" H 7400 3700 50  0001 C CNN
+F 1 "SMA_OUT" V 7510 3640 50  0000 C CNN
+F 2 "Molex_SMA:Molex_SMA_Jack_Edge_Mount" H 7400 3700 50  0001 C CNN
 F 3 "" H 7400 3700 50  0000 C CNN
 	1    7400 3700
@@
 P 7150 3350
 F 0 "C7" H 7175 3450 50  0000 L CNN
-F 1 "4,7uF" H 7175 3250 50  0000 L CNN
-F 2 "Capacitors_SMD:c_elec_5x5.3" H 7188 3200 50  0001 C CNN
+F 1 "100nF" H 7175 3250 50  0000 L CNN
+F 2 "Capacitors_SMD:C_0603_HandSoldering" H 7188 3200 50  0001 C CNN
 F 3 "" H 7150 3350 50  0000 C CNN
 	1    7150 3350
@@
 P 5200 3000
 F 0 "C4" H 5225 3100 50  0000 L CNN
-F 1 "4,7uF" H 5225 2900 50  0000 L CNN
-F 2 "Capacitors_SMD:c_elec_5x5.3" H 5238 2850 50  0001 C CNN
+F 1 "100n" H 5225 2900 50  0000 L CNN
+F 2 "Capacitors_SMD:C_0603_HandSoldering" H 5238 2850 50  0001 C CNN
 F 3 "" H 5200 3000 50  0000 C CNN
 	1    5200 3000
@@
 P 4050 3650
 F 0 "P1" H 4060 3770 50  0000 C CNN
-F 1 "BNC" V 4160 3590 50  0000 C CNN
-F 2 "" H 4050 3650 50  0001 C CNN
+F 1 "SMA_LO" V 4160 3590 50  0000 C CNN
+F 2 "Molex_SMA:Molex_SMA_Jack_Edge_Mount" H 4050 3650 50  0001 C CNN
 F 3 "" H 4050 3650 50  0000 C CNN
 	1    4050 3650
@@
 $EndComp
 $Comp
-L JUMPER3 JP1
-U 1 1 59FE12EE
-P 4350 3200
-F 0 "JP1" H 4400 3100 50  0000 L CNN
-F 1 "JUMPER3" H 4350 3300 50  0000 C BNN
-F 2 "Connect:PINHEAD1-3" H 4350 3200 50  0001 C CNN
-F 3 "" H 4350 3200 50  0000 C CNN
-	1    4350 3200
-	0    -1   -1   0
-$EndComp
-$Comp
-L GND #PWR010
-U 1 1 59FE146A
-P 4350 3450
-F 0 "#PWR010" H 4350 3200 50  0001 C CNN
-F 1 "GND" H 4350 3300 50  0000 C CNN
-F 2 "" H 4350 3450 50  0000 C CNN
-F 3 "" H 4350 3450 50  0000 C CNN
-	1    4350 3450
-	1    0    0    -1
-$EndComp
-$Comp
-L VCC #PWR011
-U 1 1 59FE149C
-P 4350 2800
-F 0 "#PWR011" H 4350 2650 50  0001 C CNN
-F 1 "VCC" H 4350 2950 50  0000 C CNN
-F 2 "" H 4350 2800 50  0000 C CNN
-F 3 "" H 4350 2800 50  0000 C CNN
-	1    4350 2800
-	1    0    0    -1
-$EndComp
-$Comp
 L TRANSFO4 T1
 U 1 1 59FE21E4
-P 5850 5200
-F 0 "T1" H 5850 5450 50  0000 C CNN
-F 1 "TRANSFO4" H 5850 4900 50  0000 C CNN
-F 2 "" H 5850 5200 50  0001 C CNN
-F 3 "" H 5850 5200 50  0000 C CNN
-	1    5850 5200
-	0    1    1    0
+P 5850 5050
+F 0 "T1" H 5850 5300 50  0000 C CNN
+F 1 "TRANSFO4" H 5850 4750 50  0000 C CNN
+F 2 "Balun:Balun" H 5850 5050 50  0001 C CNN
+F 3 "" H 5850 5050 50  0000 C CNN
+	1    5850 5050
+	0    -1   1    0
 $EndComp
 Wire Wire Line
@@
 Wire Wire Line
 	4850 3700 4850 3650
-Wire Wire Line
-	5100 3400 4700 3400
-Wire Wire Line
-	4700 3400 4700 3200
-Wire Wire Line
-	4700 3200 4450 3200
-Wire Wire Line
-	4350 2800 4350 2950
-Wire Wire Line
-	6050 4800 6050 4700
-Wire Wire Line
-	6050 4700 5900 4700
-Wire Wire Line
-	5900 4700 5900 4500
-Wire Wire Line
-	5750 4500 5750 4700
-Wire Wire Line
-	5750 4700 5650 4700
-Wire Wire Line
-	5650 4700 5650 4800
-Wire Wire Line
-	5850 4800 5850 4550
-Connection ~ 5850 4550
 $Comp
 L BNC P3
@@
 P 5950 5950
 F 0 "P3" H 5960 6070 50  0000 C CNN
-F 1 "BNC" V 6060 5890 50  0000 C CNN
-F 2 "" H 5950 5950 50  0001 C CNN
+F 1 "SMA_Q" V 6060 5890 50  0000 C CNN
+F 2 "Molex_SMA:Molex_SMA_Jack_Edge_Mount" H 5950 5950 50  0001 C CNN
 F 3 "" H 5950 5950 50  0000 C CNN
 	1    5950 5950
 	0    1    1    0
 $EndComp
-Wire Wire Line
-	5750 5950 5650 5950
-Wire Wire Line
-	5650 5950 5650 5600
-Wire Wire Line
-	5950 5800 6050 5800
-Wire Wire Line
-	6050 5800 6050 5600
-$Comp
-L GND #PWR012
+$Comp
+L GND #PWR010
 U 1 1 59FE27BD
 P 5650 5950
-F 0 "#PWR012" H 5650 5700 50  0001 C CNN
+F 0 "#PWR010" H 5650 5700 50  0001 C CNN
 F 1 "GND" H 5650 5800 50  0000 C CNN
 F 2 "" H 5650 5950 50  0000 C CNN
@@
 F 0 "T2" H 5950 2550 50  0000 C CNN
 F 1 "TRANSFO4" H 5950 2000 50  0000 C CNN
-F 2 "" H 5950 2300 50  0001 C CNN
+F 2 "Balun:Balun" H 5950 2300 50  0001 C CNN
 F 3 "" H 5950 2300 50  0000 C CNN
 	1    5950 2300
-	0    -1   -1   0
-$EndComp
-Wire Wire Line
-	5750 3050 5750 2700
-Wire Wire Line
-	5900 3050 6000 3050
-Wire Wire Line
-	6000 3050 6000 2800
-Wire Wire Line
-	6000 2800 6150 2800
-Wire Wire Line
-	6150 2800 6150 2700
-Wire Wire Line
-	5950 2700 5950 2850
-Connection ~ 5950 2850
+	0    1    -1   0
+$EndComp
 $Comp
 L BNC P2
@@
 P 5900 1600
 F 0 "P2" H 5910 1720 50  0000 C CNN
-F 1 "BNC" V 6010 1540 50  0000 C CNN
-F 2 "" H 5900 1600 50  0001 C CNN
+F 1 "SMA_I" V 6010 1540 50  0000 C CNN
+F 2 "Molex_SMA:Molex_SMA_Jack_Edge_Mount" H 5900 1600 50  0001 C CNN
 F 3 "" H 5900 1600 50  0000 C CNN
 	1    5900 1600
 	-1   0    0    -1
 $EndComp
-Wire Wire Line
-	6150 1900 6150 1600
-Wire Wire Line
-	6150 1600 6050 1600
-Wire Wire Line
-	5900 1800 5750 1800
-Wire Wire Line
-	5750 1800 5750 1900
-$Comp
-L GND #PWR013
+$Comp
+L GND #PWR011
 U 1 1 59FE2E2F
-P 5900 1800
-F 0 "#PWR013" H 5900 1550 50  0001 C CNN
-F 1 "GND" H 5900 1650 50  0000 C CNN
-F 2 "" H 5900 1800 50  0000 C CNN
-F 3 "" H 5900 1800 50  0000 C CNN
-	1    5900 1800
+P 5900 1850
+F 0 "#PWR011" H 5900 1600 50  0001 C CNN
+F 1 "GND" H 5900 1700 50  0000 C CNN
+F 2 "" H 5900 1850 50  0000 C CNN
+F 3 "" H 5900 1850 50  0000 C CNN
+	1    5900 1850
 	1    0    0    -1
 $EndComp
@@
 F 0 "L1" V 10350 3400 50  0000 C CNN
 F 1 "20uH" V 10500 3400 50  0000 C CNN
-F 2 "" H 10400 3400 50  0001 C CNN
+F 2 "Resistors_SMD:R_0805_HandSoldering" H 10400 3400 50  0001 C CNN
 F 3 "" H 10400 3400 50  0000 C CNN
 	1    10400 3400
@@
 F 0 "U1" H 9800 3254 50  0000 C CNN
 F 1 "7805" H 9650 3650 50  0000 C CNN
-F 2 "TO_SOT_Packages_SMD:TO-263-3Lead" H 9650 3450 50  0001 C CNN
+F 2 "TO_SOT_Packages_THT:TO-220_Neutral123_Vertical" H 9650 3450 50  0001 C CNN
 F 3 "" H 9650 3450 50  0000 C CNN
 	1    9650 3450
@@
 	8850 3700 10700 3700
 $Comp
-L GND #PWR014
+L GND #PWR012
 U 1 1 59FE43F2
 P 10100 3700
-F 0 "#PWR014" H 10100 3450 50  0001 C CNN
+F 0 "#PWR012" H 10100 3450 50  0001 C CNN
 F 1 "GND" H 10100 3550 50  0000 C CNN
 F 2 "" H 10100 3700 50  0000 C CNN
@@
 	4550 3850 4500 3850
 $Comp
-L VCC #PWR015
+L VCC #PWR013
 U 1 1 59FE4933
 P 10700 3350
-F 0 "#PWR015" H 10700 3200 50  0001 C CNN
+F 0 "#PWR013" H 10700 3200 50  0001 C CNN
 F 1 "VCC" H 10700 3500 50  0000 C CNN
 F 2 "" H 10700 3350 50  0000 C CNN
@@
 	8850 3400 9250 3400
 Connection ~ 9250 3700
+NoConn ~ 5100 3400
+Connection ~ 6200 3000
+Wire Wire Line
+	5750 2700 5750 3050
+Wire Wire Line
+	6150 2700 6150 2800
+Wire Wire Line
+	6150 2800 5900 2800
+Wire Wire Line
+	5900 2800 5900 3050
+Wire Wire Line
+	5950 2700 5950 3000
+Connection ~ 5950 3000
+Wire Wire Line
+	6050 1600 6150 1600
+Wire Wire Line
+	6150 1600 6150 1900
+Wire Wire Line
+	5900 1800 5900 1850
+Wire Wire Line
+	5750 1900 5750 1850
+Wire Wire Line
+	5750 1850 5900 1850
+Connection ~ 5900 1850
+Wire Wire Line
+	5650 4650 5650 4500
+Wire Wire Line
+	5650 4500 5750 4500
+Wire Wire Line
+	6050 4650 5950 4650
+Wire Wire Line
+	5950 4650 5950 4500
+Wire Wire Line
+	5950 4500 5900 4500
+Wire Wire Line
+	5850 4650 5850 4550
+Connection ~ 5850 4550
+Wire Wire Line
+	6050 5450 6050 5750
+Wire Wire Line
+	6050 5750 5950 5750
+Wire Wire Line
+	5950 5750 5950 5800
+Wire Wire Line
+	5650 5450 5650 5950
+Wire Wire Line
+	5650 5950 5750 5950
+Connection ~ 5650 5950
 $EndSCHEMATC
