File: hardware/Iq Mixer.kicad_pcb (KiCad board)
At the start: 2 copper layers, 52.4 x 46 mm, 23 parts, among them IC1 LTC5598, P1 SMA_LO, P2 SMA_I, P3 SMA_Q, P4 SMA_OUT, T1 TRANSFO4, T2 TRANSFO4, U1 7805

Commit message: Various little improvements in layout, Silkscreen Hints, Gerber generated
Parts:
- moved P3 2.54 mm to (63.2, 100.1)
- moved C11 0.76 mm to (55.1, 68.8)
- moved C7 0.51 mm to (57.4, 79.0)
Routing:
- net (no net): track 0.00 -> 6.88 mm
- net VCC: track 44.4 -> 50.5 mm
- net Net-(C9-Pad2): track 16.0 -> 22.0 mm
- net Net-(C10-Pad1): track 14.4 -> 19.5 mm
- net GND: track 38.3 -> 42.4 mm, vias 0 -> 2
- net Net-(C5-Pad2): track 14.4 -> 12.0 mm
- net Net-(P3-Pad1): track 9.06 -> 6.72 mm
Other:
- net class Default: clearance 0.2 -> 0.125
- rule trace_clearance: 0.2 -> 0.125
- board text added: "GND"
- board text added: "I Signal"
- board text added: "IQMixer-Testboard LTC5598 V1.0 11-2017 AfuJugendFdb DARC T19 Julian, DM1JZ"
- board text added: "IQMixer-Testboard V1.0 11-2017"
- board text added: "LO IN"
- board text added: "Q Signal"
- board text added: "RF OUT"
- board text added: "VCC"
